Commit message: test robot_marker

File: toy_ros_space/src/sim_drone/urdf/kaka.urdf (robot description, URDF)
Before this commit: robot kaka, 1 links, 0 joints
Links:
- added link kaka_base_link, mass 0.2; collision cylinder length=0.04 radius=0.04; visual cylinder length=0.04 radius=0.04
- added link left_arm, mass 0.07; collision box size=0.17 .01 .01; visual box size=0.17 .01 .01
- added link left_disk, mass 0.01; collision cylinder length=0.001 radius=0.1; visual cylinder length=0.001 radius=0.1
- added link right_arm, mass 0.07; collision box size=0.17 .01 .01; visual box size=0.17 .01 .01
- added link right_disk, mass 0.01; collision cylinder length=0.001 radius=0.1; visual cylinder length=0.001 radius=0.1
- link base_link: mass 0.2 -> None; geometry 
Joints:
- added joint base_to_left_arm: type revolute, parent kaka_base_link, child left_arm, origin xyz=-0.06 0 0, axis -1 0 0, limit lower=-1.57075 upper=1.57075 effort=1000.0 velocity=0.5
- added joint base_to_right_arm: type revolute, parent kaka_base_link, child right_arm, origin xyz=0.06 0 0, axis 1 0 0, limit lower=-1.57075 upper=1.57075 effort=1000.0 velocity=0.5
- added joint dummy_joint: type fixed, parent base_link, child kaka_base_link, origin xyz=0 0 0
- added joint left_disk_arm_joint: type fixed, parent left_arm, child left_disk, origin xyz=-0.085 0 0.019
- added joint right_disk_arm_joint: type fixed, parent right_arm, child right_disk, origin xyz=0.085 0 0.019

File: toy_ros_space/src/sim_drone/urdf/kaka.xacro (robot description, xacro)
@@ -42,5 +42,5 @@
       <axis xyz="${reflect} 0 0"/>
       <limit effort="1000.0" lower="-${pi/2}" upper="${pi/2}" velocity="0.5"/>
-      <parent link="base_link"/>
+      <parent link="kaka_base_link"/>
       <child link="${prefix}_arm"/>
       <origin xyz="${reflect*(width+.02)} 0 0" />
@@ -74,4 +74,6 @@
 <!-- end of macro define -->
   <link name="base_link">
+  </link>
+  <link name="kaka_base_link">
     <visual>
       <geometry>
@@ -89,4 +91,9 @@
     <xacro:default_inertial mass="0.2"/>
   </link>
+  <joint name="dummy_joint" type="fixed">
+    <parent link="base_link"/>
+    <child link="kaka_base_link"/>
+    <origin xyz="0 0 0" />
+  </joint>
   <xacro:arm prefix="right" reflect="1" />
   <xacro:arm prefix="left" reflect="-1" />

Commit message: add KAKA test launch file. Now we can use joy to control kaka parts to move

File: toy_ros_space/src/sim_drone/urdf/kaka.urdf (robot description, URDF)
Before this commit: robot kaka, 6 links, 5 joints
Links:
- removed link kaka_base_link
- link base_link: mass None -> 0.2; geometry collision cylinder length=0.04 radius=0.04; visual cylinder length=0.04 radius=0.04
Joints:
- removed joint dummy_joint
- joint base_to_left_arm: parent kaka_base_link -> base_link
- joint base_to_right_arm: parent kaka_base_link -> base_link

File: toy_ros_space/src/sim_drone/urdf/kaka.xacro (robot description, xacro)
@@ -42,5 +42,5 @@
       <axis xyz="${reflect} 0 0"/>
       <limit effort="1000.0" lower="-${pi/2}" upper="${pi/2}" velocity="0.5"/>
-      <parent link="kaka_base_link"/>
+      <parent link="base_link"/>
       <child link="${prefix}_arm"/>
       <origin xyz="${reflect*(width+.02)} 0 0" />
@@ -74,6 +74,4 @@
 <!-- end of macro define -->
   <link name="base_link">
-  </link>
-  <link name="kaka_base_link">
     <visual>
       <geometry>
@@ -91,9 +89,4 @@
     <xacro:default_inertial mass="0.2"/>
   </link>
-  <joint name="dummy_joint" type="fixed">
-    <parent link="base_link"/>
-    <child link="kaka_base_link"/>
-    <origin xyz="0 0 0" />
-  </joint>
   <xacro:arm prefix="right" reflect="1" />
   <xacro:arm prefix="left" reflect="-1" />

Commit message: fix quad height controller

File: toy_ros_space/src/sim_drone/urdf/kaka.urdf (robot description, URDF)
Before this commit: robot kaka, 5 links, 4 joints
Joints:
- joint base_to_left_arm: axis -1 0 0 -> 0 1 0; origin xyz=-0.06 0 0 -> xyz=0 0.06  0
- joint base_to_right_arm: axis 1 0 0 -> 0 -1 0; origin xyz=0.06 0 0 -> xyz=0 -0.06  0
- joint left_disk_arm_joint: origin xyz=-0.085 0 0.019 -> xyz=0 0.085 0.019
- joint right_disk_arm_joint: origin xyz=0.085 0 0.019 -> xyz=0 -0.085 0.019

File: toy_ros_space/src/sim_drone/urdf/kaka.xacro (robot description, xacro)
@@ -40,9 +40,9 @@
     </link>
     <joint name="base_to_${prefix}_arm" type="revolute">
-      <axis xyz="${reflect} 0 0"/>
+      <axis xyz="0 ${reflect} 0"/>
       <limit effort="1000.0" lower="-${pi/2}" upper="${pi/2}" velocity="0.5"/>
       <parent link="base_link"/>
       <child link="${prefix}_arm"/>
-      <origin xyz="${reflect*(width+.02)} 0 0" />
+      <origin xyz="0 ${reflect*(width+.02)}  0" />
     </joint>
     <link name="${prefix}_disk">
@@ -67,5 +67,5 @@
       <parent link="${prefix}_arm"/>
       <child link="${prefix}_disk"/>
-      <origin xyz="${reflect*armlen/2} 0 0.019" />
+      <origin xyz="0 ${reflect*armlen/2} 0.019" />
     </joint>
   </xacro:macro>
@@ -89,5 +89,5 @@
     <xacro:default_inertial mass="0.2"/>
   </link>
-  <xacro:arm prefix="right" reflect="1" />
-  <xacro:arm prefix="left" reflect="-1" />
+  <xacro:arm prefix="right" reflect="-1" />
+  <xacro:arm prefix="left" reflect="1" />
 </robot>
